File: hardware/v1.1/teensythumbboard.kicad_pcb (KiCad board)
At the start: 2 copper layers, 97.2 x 81.3 mm, 79 parts, among them J1 Conn_01x01, J2 Conn_01x01, J3 Conn_01x01, J4 Conn_01x01, J5 Conn_01x08_Male, J6 Conn_01x01_Male, J7 Conn_01x01_Male, J8 Conn_01x01_Male, SW1 SW_Push, SW10 SW_Push, SW11 SW_Push, SW12 SW_Push, SW13 SW_Push, SW14 SW_Push, SW15 SW_Push, SW16 SW_Push, SW17 SW_Push, SW18 SW_Push, SW19 SW_Push, SW2 SW_Push, SW20 SW_Push, SW21 SW_Push, SW22 SW_Push, SW23 SW_Push, SW24 SW_Push, SW25 SW_Push, SW26 SW_Push, SW27 SW_Push, SW28 SW_Push, SW29 SW_Push, SW3 SW_Push, SW30 SW_Push, SW31 SW_Push, SW32 SW_Push, SW33 SW_Push, SW34 SW_Push, SW35 SW_Push, SW36 SW_Push, SW37 SW_Push, SW38 SW_Push, SW39 SW_Push, SW4 SW_Push, SW40 SW_Push, SW41 SW_Push, SW42 SW_Push, SW43 SW_Push, SW44 SW_Push, SW45 SW_Push, SW46 SW_Push, SW47 SW_Push, SW48 SW_Push, SW49 SW_Push, SW5 SW_Push, SW50 SW_Push, SW51 SW_Push, SW52 SW_Push, SW53 SW_Push, SW54 SW_Push, SW55 SW_Push, SW56 SW_Push, SW57 SW_Push, SW58 SW_Push, SW59 SW_Push, SW6 SW_Push, SW60 SW_Push, SW7 SW_Push, SW8 SW_Push, SW9 SW_Push, U1 Teensy3.2

Commit message: Add v1.1 kicad project
Parts:
- removed J6, J8: Conn_01x01_Male, teensy32:PinHeader_1x01_P2.54mm_Vertical
- U1: footprint teensy32:Teensy32 -> teensy32:Teensy32_InnerProto
- moved D10 0.54 mm to (161.4, 76.2)
Connections:
- U1 pad 15: (no net) -> Net-(U1-Pad15)
- U1 pad 16: (no net) -> Net-(U1-Pad16)
- U1 pad 18: (no net) -> Net-(U1-Pad18)
- U1 pad 19: (no net) -> Net-(U1-Pad19)
- U1 pad 32: (no net) -> Net-(U1-Pad32)
- U1 pad 34: (no net) -> Net-(U1-Pad34)
- U1 pad 35: (no net) -> Net-(U1-Pad35)
- U1 pad 36: (no net) -> Net-(U1-Pad36)
- U1 pad 37: (no net) -> Net-(U1-Pad37)
Routing:
- net GND: track 0.00 -> 18.2 mm, vias 2 -> 7
- net SDA: track 39.7 -> 57.4 mm, vias 0 -> 1
- net SCL: track 37.1 -> 52.9 mm, vias 0 -> 1
- net ROW1: track 188.7 -> 197.8 mm
- net SCK: track 54.2 -> 62.4 mm
- net COL0: track 37.8 -> 42.4 mm, vias 1 -> 2
- net 22-A8: track 35.8 -> 31.6 mm, vias 1 -> 0
- net ROW0: track 233.7 -> 237.5 mm
- net COL7: track 48.8 -> 51.6 mm
- net ROW2: track 193.5 -> 196.0 mm
- net Net-(U1-Pad32): track 0.00 -> 2.54 mm
- net Net-(U1-Pad19): track 0.00 -> 2.54 mm
- net Net-(U1-Pad18): track 0.00 -> 2.54 mm
- net Net-(U1-Pad16): track 0.00 -> 2.54 mm
- net Net-(U1-Pad15): track 0.00 -> 2.54 mm
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Other:
- board text added: "Teensy Thumb Board v1.1"
- board text added: "github.com/ AnthonyDiGirolamo"
- board text removed: "3.3v"
- board text removed: "A10"
- board text removed: "A10-D22"
- board text removed: "A11"
- board text removed: "A11-D21"
- board text removed: "A12"
- board text removed: "A13"
- board text removed: "A14"
- board text removed: "A9/D32"
- board text removed: "AREF"
- board text removed: "AREF-D23"
- board text removed: "D24"
- board text removed: "D25"
- board text removed: "D26"
- board text removed: "D27"
- board text removed: "D28"
- board text removed: "D29"
- board text removed: "D30"
- board text removed: "D31"
- board text removed: "D32"
- board text removed: "D33"
- board text removed: "GND"
- board text removed: "Prg"
- board text removed: "Teensy 3.2"
- board text removed: "Teensy Thumb Board 1.0"
- board text removed: "VUSB-AGND"
- board text removed: "Vbat"
- board text removed: "Vin"
