File: hardware/v1.1/teensythumbboard.sch (KiCad schematic (older format))
At the start: 79 parts, among them J1 Conn_01x01, J2 Conn_01x01, J3 Conn_01x01, J4 Conn_01x01, J5 Conn_01x08_Male, J6 Conn_01x01_Male, J7 Conn_01x01_Male, J8 Conn_01x01_Male, SW1 SW_Push, SW10 SW_Push, SW11 SW_Push, SW12 SW_Push, SW13 SW_Push, SW14 SW_Push, SW15 SW_Push, SW16 SW_Push, SW17 SW_Push, SW18 SW_Push, SW19 SW_Push, SW2 SW_Push, SW20 SW_Push, SW21 SW_Push, SW22 SW_Push, SW23 SW_Push, SW24 SW_Push, SW25 SW_Push, SW26 SW_Push, SW27 SW_Push, SW28 SW_Push, SW29 SW_Push, SW3 SW_Push, SW30 SW_Push, SW31 SW_Push, SW32 SW_Push, SW33 SW_Push, SW34 SW_Push, SW35 SW_Push, SW36 SW_Push, SW37 SW_Push, SW38 SW_Push, SW39 SW_Push, SW4 SW_Push, SW40 SW_Push, SW41 SW_Push, SW42 SW_Push, SW43 SW_Push, SW44 SW_Push, SW45 SW_Push, SW46 SW_Push, SW47 SW_Push, SW48 SW_Push, SW49 SW_Push, SW5 SW_Push, SW50 SW_Push, SW51 SW_Push, SW52 SW_Push, SW53 SW_Push, SW54 SW_Push, SW55 SW_Push, SW56 SW_Push, SW57 SW_Push, SW58 SW_Push, SW59 SW_Push, SW6 SW_Push, SW60 SW_Push, SW7 SW_Push, SW8 SW_Push, SW9 SW_Push, U1 Teensy3.2

Commit message: Add v1.1 kicad project
Parts:
- U1: footprint teensy32:Teensy32 -> teensy32:Teensy32_InnerProto; symbol teensythumbboard-rescue:Teensy3.2-teensy32 -> teensy32:Teensy3.2
Changed lines of the file:
@@
 Title "Teensy Thumb Board"
 Date "2018-11-11"
-Rev "1.0"
+Rev "1.1"
 Comp ""
 Comment1 ""
@@
 $EndComp
 $Comp
-L teensythumbboard-rescue:Teensy3.2-teensy32 U1
+L teensy32:Teensy3.2 U1
 U 1 1 5B82F09B
 P 3400 6200
 F 0 "U1" H 3400 7787 60  0000 C CNN
 F 1 "Teensy3.2" H 3400 7681 60  0000 C CNN
-F 2 "teensy32:Teensy32" H 3400 5400 60  0001 C CNN
+F 2 "teensy32:Teensy32_InnerProto" H 3400 5400 60  0001 C CNN
 F 3 "" H 3400 5400 60  0000 C CNN
 	1    3400 6200
